File: STM32_Clone.kicad_pcb (KiCad board)
At the start: 2 copper layers, 37 x 31.5 mm, 32 parts, among them J1 USB_B_Micro, J2 Conn_01x04_Male, J3 Conn_01x04_Male, J4 Conn_01x04_Male, SW1 SW_SPDT, U1 AMS1117-3.3, U2 STM32F103C8T6, Y1 16MHz

Commit message: Update README.md
Other:
- net class Default removed
